File: hardware/GamepadPMOD/GamepadPMOD.kicad_sch (KiCad schematic)
At the start: 23 parts, among them J1 SFC connector VERT, J2 SFC connector VERT, J3 10129382-912001BLF, J4 613012243121, J5 Conn_02x03_Odd_Even, SW1 434121025816, U1 CH32V003F4U6

Commit message: Specify red status LED part
Co-authored-by: Copilot <223556219+Copilot@users.noreply.github.com>
Parts:
- D1: Characteristics LED orange -> Red 630nm, 1.95V typical at 20mA, cathode pad 1; DigikeyPN (none) -> 754-1123-1-ND; LCSC C965800 -> (none); MPN (none) -> APT1608SURCK
Changed lines of the file:
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@@
 			)
 		)
-		(property "Datasheet" ""
+		(property "Datasheet" "https://www.kingbrightusa.com/images/catalog/SPEC/APT1608SURCK.pdf"
 			(at 53.34 68.58 0)
 			(hide yes)
@@
 			)
 		)
-		(property "Description" "Light emitting diode"
+		(property "Description" "Kingbright red LED, 630 nm, 0603 (1608 metric), clear lens"
 			(at 53.34 68.58 0)
 			(hide yes)
@@
 			)
 		)
-		(property "Characteristics" "LED orange"
+		(property "Characteristics" "Red 630nm, 1.95V typical at 20mA, cathode pad 1"
 			(at 53.34 68.58 0)
 			(hide yes)
@@
 			)
 		)
-		(property "MPN" ""
+		(property "MPN" "APT1608SURCK"
 			(at 53.34 68.58 0)
 			(hide yes)
@@
 			)
 		)
-		(property "DigikeyPN" ""
+		(property "DigikeyPN" "754-1123-1-ND"
 			(at 53.34 68.58 0)
 			(hide yes)
@@
 			)
 		)
-		(property "LCSC" "C965800"
+		(property "LCSC" ""
 			(at 53.34 68.58 0)
 			(hide yes)
